File: Thermistor_readout.brd (EAGLE design)
At the start: 59.4 x 43.2 mm, 22 parts, among them Q1 BC550C, U1 TI_NATIONAL_SEMICONDUCTOR_LF3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, U2 TI_NATIONAL_SEMICONDUCTOR_LF3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, U3 ANALOG_DEVICES_ADG725BSUZANAL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, U4 TI_NATIONAL_SEMICONDUCTOR_LF3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

Commit message: New_Re_size
Parts:
- RE: device 1AKarstenLib:R0805H -> 1AKarstenLib:R1206H
- moved RE 93.5 mm to (0.00, -44.5), turned to 0 degrees
Changed lines of the file:
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@@
 <element name="R6" library="1AKarstenLib" package="R0805H" value="20kΩ" x="49.53" y="12.7"/>
 <element name="R7" library="1AKarstenLib" package="R0805H" value="20kΩ" x="38.1" y="26.67"/>
-<element name="RE" library="1AKarstenLib" package="R0805H" value="" x="55.88" y="30.48" rot="R90"/>
 <element name="U2" library="TI National Semiconductor - LF356M" package="TI_NATIONAL_SEMICONDUCTOR_LF356M_2" value="TI_NATIONAL_SEMICONDUCTOR_LF356MTI_NATIONAL_SEMICONDUCTOR_LF356M_0_2" x="49.53" y="20.32">
 <attribute name="VAULT_GUID" value="86B7F69C-A366-49BF-B4AD-C30E98E1479F" x="49.53" y="20.32" size="1.778" layer="27" display="off"/>
@@
 <element name="C7" library="1AKarstenLib" package="R0805H" value="" x="0" y="-31.75"/>
 <element name="C8" library="1AKarstenLib" package="R0805H" value="" x="0" y="-38.1"/>
+<element name="RE" library="1AKarstenLib" package="R1206H" value="" x="0" y="-44.45"/>
 </elements>
 <signals>
@@
 <contactref element="Q1" pad="E"/>
 <contactref element="RE" pad="2"/>
-<wire x1="52.07" y1="31.75" x2="55.88" y2="31.623" width="0" layer="19" extent="1-1"/>
+<wire x1="1.6002" y1="-44.45" x2="52.07" y2="31.75" width="0" layer="19" extent="1-1"/>
 </signal>
 <signal name="N$24">
@@
 <signal name="GND">
 <contactref element="R2" pad="1"/>
-<contactref element="RE" pad="1"/>
 <contactref element="R7" pad="1"/>
 <contactref element="U3" pad="24"/>
@@
 <contactref element="C8" pad="2"/>
 <contactref element="C7" pad="1"/>
-<wire x1="-1.143" y1="-31.75" x2="1.143" y2="-38.1" width="0" layer="19" extent="1-1"/>
-<wire x1="1.143" y1="-19.05" x2="-1.143" y2="-31.75" width="0" layer="19" extent="1-1"/>
-<wire x1="-1.143" y1="-12.7" x2="1.143" y2="-19.05" width="0" layer="19" extent="1-1"/>
-<wire x1="15.367" y1="22.86" x2="-1.143" y2="-12.7" width="0" layer="19" extent="1-1"/>
+<contactref element="RE" pad="1"/>
+<wire x1="48.133" y1="25.4" x2="57.023" y2="20.955" width="0" layer="19" extent="1-1"/>
+<wire x1="36.957" y1="26.67" x2="48.133" y2="25.4" width="0" layer="19" extent="1-1"/>
+<wire x1="39.497" y1="13.97" x2="36.957" y2="26.67" width="0" layer="19" extent="1-1"/>
+<wire x1="41.91" y1="5.08" x2="39.497" y2="13.97" width="0" layer="19" extent="1-1"/>
+<wire x1="23.79" y1="19.34" x2="36.957" y2="26.67" width="0" layer="19" extent="1-1"/>
+<wire x1="23.79" y1="18.84" x2="23.79" y2="19.34" width="0" layer="19" extent="1-1"/>
+<wire x1="15.367" y1="22.86" x2="23.79" y2="19.34" width="0" layer="19" extent="1-1"/>
+<wire x1="15.367" y1="25.4" x2="15.367" y2="22.86" width="0" layer="19" extent="1-1"/>
+<wire x1="-1.143" y1="-12.7" x2="15.367" y2="22.86" width="0" layer="19" extent="1-1"/>
+<wire x1="1.143" y1="-19.05" x2="-1.143" y2="-12.7" width="0" layer="19" extent="1-1"/>
+<wire x1="-1.143" y1="-31.75" x2="1.143" y2="-19.05" width="0" layer="19" extent="1-1"/>
+<wire x1="1.143" y1="-38.1" x2="-1.143" y2="-31.75" width="0" layer="19" extent="1-1"/>
+<wire x1="-1.6002" y1="-44.45" x2="1.143" y2="-38.1" width="0" layer="19" extent="1-1"/>
 </signal>
 <signal name="+5V">

Commit message: First_PCB_tentative
Parts:
- moved RE 85.2 mm to (51.4, 23.5), turned to 180 degrees
- moved C6 84.7 mm to (71.8, 26.0)
- moved C8 81.9 mm to (66.7, 9.53)
- moved U4 65.6 mm to (59.7, 8.89)
- moved C5 64.9 mm to (55.9, 20.3)
- moved U1 64.3 mm to (59.7, 25.4)
- moved C7 63.5 mm to (50.8, 6.35)
- moved C4 33.9 mm to (22.9, 13.3)
- moved U2 33.2 mm to (16.5, 17.1), turned to 270 degrees
- moved C3 31.0 mm to (10.2, 19.7)
- moved R6 22.8 mm to (27.3, 17.8)
- moved R7 19.8 mm to (18.4, 24.8), turned to 180 degrees
- moved R1 17.7 mm to (36.8, 19.1), turned to 180 degrees
- moved R4 16.8 mm to (51.4, 27.9), turned to 180 degrees
- moved R5 9.67 mm to (41.9, 14.0), turned to 180 degrees
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Routing:
- net +5V: track 0.00 -> 143.9 mm, vias 0 -> 2
- net +15V: track 0.00 -> 95.7 mm
- net -15V: track 0.00 -> 76.5 mm, vias 0 -> 2
- net N$13: track 0.00 -> 44.1 mm
- net N$14: track 0.00 -> 43.2 mm
- net N$11: track 0.00 -> 42.2 mm
- net C$14: track 0.00 -> 39.3 mm, vias 0 -> 2
- net N$5: track 0.00 -> 35.0 mm
- net C$1: track 0.00 -> 33.0 mm
- net C$13: track 0.00 -> 30.3 mm, vias 0 -> 2
- net C$2: track 0.00 -> 30.1 mm
- net N$4: track 0.00 -> 28.0 mm, vias 0 -> 2
- net C$3: track 0.00 -> 27.8 mm
- net C$15: track 0.00 -> 25.8 mm
- net C$4: track 0.00 -> 25.7 mm
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Other:
- board size 59.4 x 43.2 mm -> 75.9 x 43.2 mm

Commit message: Simil_complete1
Routing:
- net N$3: track 0.00 -> 50.8 mm, vias 0 -> 2
- net N$6: track 15.2 -> 63.0 mm, vias 2 -> 4
- net C$16: track 0.00 -> 27.1 mm, vias 0 -> 2
- net N$8: track 0.00 -> 22.4 mm, vias 0 -> 2
- net C$15: track 25.8 -> 36.5 mm, vias 0 -> 2
- net N$2: track 0.00 -> 6.45 mm
Changed lines of the file:
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@@
 <param name="TopRouterVariant" value="0"/>
 <param name="tpViaShape" value="round"/>
-<param name="PrefDir.1" value="a"/>
+<param name="PrefDir.1" value="*"/>
 <param name="PrefDir.2" value="0"/>
 <param name="PrefDir.3" value="0"/>
@@
 <param name="PrefDir.14" value="0"/>
 <param name="PrefDir.15" value="0"/>
-<param name="PrefDir.16" value="a"/>
+<param name="PrefDir.16" value="-"/>
 <param name="cfVia" value="8"/>
 <param name="cfNonPref" value="5"/>
@@
 <contactref element="Q1" pad="E"/>
 <contactref element="RE" pad="2"/>
-<wire x1="44.45" y1="22.225" x2="49.8348" y2="23.495" width="0" layer="19" extent="1-1"/>
+<wire x1="49.8348" y1="22.606" x2="49.8348" y2="23.495" width="0.254" layer="1"/>
+<wire x1="49.4792" y1="22.2504" x2="49.8348" y2="22.606" width="0.254" layer="1"/>
+<wire x1="44.45" y1="22.2504" x2="49.4792" y2="22.2504" width="0.254" layer="1"/>
+<wire x1="44.45" y1="22.2504" x2="44.45" y2="22.225" width="0.254" layer="1"/>
 </signal>
 <signal name="N$24">
@@
 <contactref element="C7" pad="1"/>
 <contactref element="RE" pad="1"/>
+<wire x1="25.0952" y1="24.384" x2="25.0600125" y2="24.3636" width="0.254" layer="1"/>
+<wire x1="25.0952" y1="24.384" x2="25.06" y2="24.42" width="0.254" layer="1"/>
+<wire x1="31.6992" y1="21.2344" x2="31.690465625" y2="21.1386" width="0.254" layer="1"/>
+<wire x1="49.657" y1="6.35" x2="41.91" y2="5.08" width="0" layer="19" extent="1-1"/>
 <wire x1="25.06" y1="23.92" x2="24.003" y2="13.335" width="0" layer="19" extent="1-1"/>
+<wire x1="46.863" y1="19.05" x2="49.657" y2="6.35" width="0" layer="19" extent="1-1"/>
 </signal>
 <signal name="+5V">
@@
 <wire x1="45.72" y1="40.005" x2="48.26" y2="37.465" width="0.254" layer="16"/>
 <wire x1="33.36" y1="27.92" x2="38.715" y2="27.92" width="0.254" layer="1"/>
-<wire x1="38.715" y1="27.92" x2="42.545" y2="27.94" width="0.254" layer="1"/>
+<wire x1="38.715" y1="27.92" x2="40.640053125" y2="27.930053125" width="0.254" layer="1"/>
+<wire x1="40.640053125" y1="27.930053125" x2="42.545" y2="27.94" width="0.254" layer="1"/>
 <wire x1="42.545" y1="27.94" x2="48.26" y2="33.655" width="0.254" layer="1"/>
 <wire x1="48.26" y1="33.655" x2="48.26" y2="37.465" width="0.254" layer="1"/>
 <wire x1="33.36" y1="24.92" x2="34.44875" y2="24.92375" width="0.254" layer="1"/>
-<wire x1="33.36" y1="24.92" x2="33.36" y2="27.92" width="0" layer="19" extent="1-1"/>
+<wire x1="33.36" y1="24.92" x2="35.40125" y2="24.92375" width="0.254" layer="1"/>
+<wire x1="35.40125" y1="24.92375" x2="37.7825" y2="23.33625" width="0.254" layer="1"/>
+<via x="37.7825" y="23.33625" extent="1-16" drill="0.6"/>
+<wire x1="37.7825" y1="23.33625" x2="37.94125" y2="25.0825" width="0.254" layer="16"/>
+<wire x1="37.94125" y1="25.0825" x2="40.48125" y2="27.14625" width="0.254" layer="16"/>
+<via x="40.48125" y="27.14625" extent="1-16" drill="0.6"/>
+<wire x1="40.48125" y1="27.14625" x2="40.640053125" y2="27.930053125" width="0.254" layer="1"/>
 </signal>
 <signal name="C$16">
@@
 <contactref element="U3" pad="40"/>
 <contactref element="Q1" pad="C"/>
-<wire x1="44.45" y1="27.305" x2="48.26" y2="40.005" width="0" layer="19" extent="1-1"/>
-<wire x1="33.36" y1="25.42" x2="44.45" y2="27.305" width="0" layer="19" extent="1-1"/>
+<wire x1="44.45" y1="29.1592" x2="44.45" y2="27.305" width="0.254" layer="1"/>
+<wire x1="48.7172" y1="33.4264" x2="44.45" y2="29.1592" width="0.254" layer="1"/>
+<wire x1="48.7172" y1="36.3728" x2="48.7172" y2="33.4264" width="0.254" layer="1"/>
+<wire x1="49.4792" y1="37.1348" x2="48.7172" y2="36.3728" width="0.254" layer="1"/>
+<wire x1="49.4792" y1="38.7604" x2="49.4792" y2="37.1348" width="0.254" layer="1"/>
+<wire x1="48.26" y1="39.9796" x2="49.4792" y2="38.7604" width="0.254" layer="1"/>
+<wire x1="48.26" y1="39.9796" x2="48.26" y2="40.005" width="0.254" layer="1"/>
+<wire x1="33.36" y1="25.42" x2="38.1" y2="25.4" width="0.254" layer="1"/>
+<wire x1="38.1" y1="25.4" x2="38.89375" y2="24.92375" width="0.254" layer="1"/>
+<via x="38.89375" y="24.92375" extent="1-16" drill="0.6"/>
+<wire x1="38.89375" y1="24.92375" x2="42.06875" y2="26.9875" width="0.254" layer="16"/>
+<via x="42.06875" y="26.9875" extent="1-16" drill="0.6"/>
+<wire x1="42.06875" y1="26.9875" x2="44.45" y2="27.305" width="0.254" layer="1"/>
 </signal>
 <signal name="N$5">
@@
 <via x="15.875" y="22.86" extent="1-16" drill="0.6"/>
 <wire x1="15.875" y1="22.86" x2="15.875" y2="19.97" width="0.254" layer="1"/>
-<wire x1="26.162" y1="17.78" x2="50.292" y2="27.94" width="0" layer="19" extent="1-1"/>
+<wire x1="50.292" y1="26.2128" x2="50.292" y2="27.94" width="0.254" layer="1"/>
+<wire x1="50.292" y1="25.0444" x2="50.292" y2="26.2128" width="0.254" layer="16"/>
+<wire x1="41.656" y1="16.4084" x2="50.292" y2="25.0444" width="0.254" layer="16"/>
+<wire x1="41.656" y1="14.986" x2="41.656" y2="16.4084" width="0.254" layer="1"/>
+<wire x1="41.7576" y1="14.8844" x2="41.656" y2="14.986" width="0.254" layer="1"/>
+<wire x1="41.7576" y1="12.8524" x2="41.7576" y2="14.8844" width="0.254" layer="1"/>
+<wire x1="26.3652" y1="12.8524" x2="41.7576" y2="12.8524" width="0.254" layer="1"/>
+<wire x1="20.4216" y1="18.796" x2="26.3652" y2="12.8524" width="0.254" layer="1"/>
+<wire x1="16.7132" y1="18.796" x2="20.4216" y2="18.796" width="0.254" layer="1"/>
+<wire x1="15.9004" y1="19.6088" x2="16.7132" y2="18.796" width="0.254" layer="1"/>
+<wire x1="15.9004" y1="19.8628" x2="15.9004" y2="19.6088" width="0.254" layer="1"/>
+<wire x1="15.9004" y1="19.8628" x2="15.875" y2="19.97" width="0.254" layer="1"/>
+<via x="50.292" y="26.2128" extent="1-16" drill="0.6096"/>
+<via x="41.656" y="16.4084" extent="1-16" drill="0.6096"/>
 </signal>
 <signal name="N$13">
@@
 <contactref element="U4" pad="2"/>
 <contactref element="R5" pad="1"/>
-<wire x1="56.865" y1="9.525" x2="62.515" y2="8.255" width="0" layer="19" extent="1-1"/>
-<wire x1="43.053" y1="13.97" x2="56.865" y2="9.525" width="0" layer="19" extent="1-1"/>
+<wire x1="43.0784" y1="13.0556" x2="43.0784" y2="13.97" width="0.254" layer="1"/>
+<wire x1="44.704" y1="11.43" x2="43.0784" y2="13.0556" width="0.254" layer="1"/>
+<wire x1="51.4604" y1="11.43" x2="44.704" y2="11.43" width="0.254" layer="1"/>
+<wire x1="51.5112" y1="11.3792" x2="51.4604" y2="11.43" width="0.254" layer="16"/>
+<wire x1="53.34" y1="11.3792" x2="51.5112" y2="11.3792" width="0.254" layer="16"/>
+<wire x1="54.0512" y1="11.3792" x2="53.34" y2="11.3792" width="0.254" layer="1"/>
+<wire x1="55.88" y1="9.5504" x2="54.0512" y2="11.3792" width="0.254" layer="1"/>
+<wire x1="56.8452" y1="9.5504" x2="55.88" y2="9.5504" width="0.254" layer="1"/>
+<wire x1="43.0784" y1="13.97" x2="43.053" y2="13.97" width="0.254" layer="1"/>
+<wire x1="56.8452" y1="9.5504" x2="56.865" y2="9.525" width="0.254" layer="1"/>
+<wire x1="59.1312" y1="8.2804" x2="62.484" y2="8.2804" width="0.254" layer="1"/>
+<wire x1="57.8612" y1="9.5504" x2="59.1312" y2="8.2804" width="0.254" layer="1"/>
+<wire x1="56.9468" y1="9.5504" x2="57.8612" y2="9.5504" width="0.254" layer="1"/>
+<wire x1="62.484" y1="8.2804" x2="62.515" y2="8.255" width="0.254" layer="1"/>
+<wire x1="56.9468" y1="9.5504" x2="56.865" y2="9.525" width="0.254" layer="1"/>
+<via x="51.4604" y="11.43" extent="1-16" drill="0.6096"/>
+<via x="53.34" y="11.3792" extent="1-16" drill="0.6096"/>
 </signal>
 <signal name="N$3">
 <contactref element="U4" pad="3"/>
 <contactref element="U3" pad="41"/>
-<wire x1="33.36" y1="25.92" x2="56.865" y2="8.255" width="0" layer="19" extent="1-1"/>
+<wire x1="57.7596" y1="8.2804" x2="56.896" y2="8.2804" width="0.254" layer="1"/>
+<wire x1="58.166" y1="7.874" x2="57.7596" y2="8.2804" width="0.254" layer="1"/>
+<wire x1="58.166" y1="6.2484" x2="58.166" y2="7.874" width="0.254" layer="1"/>
+<wire x1="55.5752" y1="3.6576" x2="58.166" y2="6.2484" width="0.254" layer="1"/>
+<wire x1="50.0888" y1="3.6576" x2="55.5752" y2="3.6576" width="0.254" layer="1"/>
+<wire x1="47.4472" y1="6.2992" x2="50.0888" y2="3.6576" width="0.254" layer="1"/>
+<wire x1="47.4472" y1="8.6868" x2="47.4472" y2="6.2992" width="0.254" layer="1"/>
+<wire x1="47.498" y1="8.7376" x2="47.4472" y2="8.6868" width="0.254" layer="1"/>
+<wire x1="47.498" y1="10.5664" x2="47.498" y2="8.7376" width="0.254" layer="1"/>
+<wire x1="45.7708" y1="12.2936" x2="47.498" y2="10.5664" width="0.254" layer="16"/>
+<wire x1="45.7708" y1="13.5128" x2="45.7708" y2="12.2936" width="0.254" layer="1"/>
+<wire x1="41.4528" y1="17.8308" x2="45.7708" y2="13.5128" width="0.254" layer="1"/>
+<wire x1="37.2872" y1="17.8308" x2="41.4528" y2="17.8308" width="0.254" layer="1"/>
+<wire x1="36.8808" y1="18.2372" x2="37.2872" y2="17.8308" width="0.254" layer="1"/>
+<wire x1="36.8808" y1="20.4216" x2="36.8808" y2="18.2372" width="0.254" layer="1"/>
+<wire x1="33.3756" y1="25.908" x2="34.3916" y2="25.908" width="0.254" layer="1"/>
+<wire x1="56.896" y1="8.2804" x2="56.865" y2="8.255" width="0.254" layer="1"/>
+<wire x1="33.3756" y1="25.908" x2="33.36" y2="25.92" width="0.254" layer="1"/>
+<via x="47.498" y="10.5664" extent="1-16" drill="0.6096"/>
+<via x="45.7708" y="12.2936" extent="1-16" drill="0.6096"/>
+<wire x1="34.3916" y1="25.908" x2="39.52875" y2="25.87625" width="0.254" layer="1"/>
+<wire x1="39.52875" y1="25.87625" x2="40.64" y2="25.0825" width="0.254" layer="1"/>
+<wire x1="40.64" y1="25.0825" x2="40.3225" y2="24.4475" width="0.254" layer="1"/>
+<wire x1="40.3225" y1="24.4475" x2="39.84625" y2="23.97125" width="0.254" layer="1"/>
+<wire x1="39.84625" y1="23.97125" x2="39.37" y2="23.33625" width="0.254" layer="1"/>
+<wire x1="39.37" y1="23.33625" x2="39.37" y2="22.38375" width="0.254" layer="1"/>
+<wire x1="39.37" y1="22.38375" x2="36.8808" y2="20.4216" width="0.254" layer="1"/>
 </signal>
 </signals>

Commit message: finished_1st_version
Routing:
- net C$12: track 22.7 -> 31.3 mm, vias 0 -> 2
- net N$3: track 50.8 -> 43.7 mm
- net GND: track 0.19 -> 0.59 mm, vias 0 -> 4

Commit message: No_error_v1
Routing:
- net -15V: track 76.5 -> 78.2 mm
- net N$24: track 21.5 -> 23.1 mm
- net +15V: track 95.7 -> 97.2 mm
- net N$4: track 28.0 -> 28.8 mm
- net N$7: track 23.6 -> 24.4 mm
