File: Thermistor_readout.sch (EAGLE design)
At the start: 25 parts, among them Q1 BC550C, U1 TI_NATIONAL_SEMICONDUCTOR_LF3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, U2 TI_NATIONAL_SEMICONDUCTOR_LF3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, U3 ANALOG_DEVICES_ADG725BSUZANAL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, U4 TI_NATIONAL_SEMICONDUCTOR_LF3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

Commit message: Re_0805_size
Parts:
- RE: device 1AKarstenLib:R-EU_SMD1206H -> 1AKarstenLib:R-EU_SMD0805H
Changed lines of the file:
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@@
 <part name="P-2" library="supply1" deviceset="-15V" device=""/>
 <part name="GND14" library="supply1" deviceset="GND" device=""/>
-<part name="RE" library="1AKarstenLib" deviceset="R-EU_SMD" device="1206H"/>
 <part name="GND15" library="supply1" deviceset="GND" device=""/>
 <part name="GND16" library="supply1" deviceset="GND" device=""/>
@@
 <part name="C11" library="1AKarstenLib" deviceset="C-EU_SMD" device="C1206H/D"/>
 <part name="CON1" library="con-harting" deviceset="CON16L" device=""/>
+<part name="RE" library="1AKarstenLib" deviceset="R-EU_SMD" device="0805H"/>
 </parts>
 <sheets>
@@
 <instance part="P-2" gate="1" x="132.08" y="66.04"/>
 <instance part="GND14" gate="1" x="152.4" y="71.12" rot="R90"/>
-<instance part="RE" gate="G$1" x="53.34" y="71.12" rot="R90"/>
 <instance part="GND15" gate="1" x="205.74" y="30.48" rot="R180"/>
 <instance part="GND16" gate="1" x="160.02" y="50.8" rot="R180"/>
@@
 <instance part="C11" gate="G$1" x="162.56" y="25.4"/>
 <instance part="CON1" gate="G$1" x="185.42" y="25.4"/>
+<instance part="RE" gate="G$1" x="53.34" y="71.12" rot="R90"/>
 </instances>
 <busses>
